File: schem/test.sch (KiCad schematic (older format))
At the start: 24 parts, among them U1 STM32F103C8

Commit message: Keys added
Parts:
- removed KEY?: IR4426, symbol IR4426
- removed P?: engine_1, ~, symbol CONN_2
- added D? (x8): DIODE, ~, symbol DIODE
- added KEY?: IR4426, symbol IR4426
- added P?: engine_1, ~, symbol CONN_2
Connections:
- wire segments 96 -> 116
Other:
- moved on the sheet: P?
Changed lines of the file:
@@
 Sheet 1 1
 Title "WebDroid  Neuraxis"
-Date "28 sep 2013"
+Date "29 sep 2013"
 Rev ""
 Comp "BSUIR 2013"
@@
 Comment4 ""
 $EndDescr
-$Comp
-L STM32F103C8 U1
-U 1 1 52384296
-P 4200 3150
-F 0 "U1" H 3300 4300 60  0000 C CNN
-F 1 "STM32F103C8" H 4150 3400 60  0000 C CNN
-F 2 "" H 4200 3150 60  0000 C CNN
-F 3 "" H 4200 3150 60  0000 C CNN
-	1    4200 3150
-	1    0    0    -1
-$EndComp
 $Comp
 L VDD #PWR01
@@
 $Comp
 L IR4426 KEY?
-U 1 1 524767BD
-P 2550 6350
-F 0 "KEY?" H 2600 6150 60  0000 C CNN
-F 1 "IR4426" H 2550 6650 60  0000 C CNN
-F 2 "" H 2600 6400 60  0000 C CNN
-F 3 "" H 2600 6400 60  0000 C CNN
-	1    2550 6350
-	1    0    0    -1
-$EndComp
-$Comp
-L IR4426 KEY?
 U 1 1 524767C3
 P 2550 7150
@@
 $Comp
 L VSS #PWR?
-U 1 1 524767CF
-P 2050 6350
-F 0 "#PWR?" H 2050 6350 30  0001 C CNN
-F 1 "VSS" H 2050 6280 30  0000 C CNN
-F 2 "" H 2050 6350 60  0000 C CNN
-F 3 "" H 2050 6350 60  0000 C CNN
-	1    2050 6350
-	1    0    0    -1
-$EndComp
-$Comp
-L VSS #PWR?
 U 1 1 524767D5
 P 2050 7150
@@
 Wire Wire Line
 	8450 1350 8600 1350
-$Comp
-L IR4426 KEY?
-U 1 1 5247734B
-P 2050 1300
-F 0 "KEY?" H 2100 1100 60  0000 C CNN
-F 1 "IR4426" H 2050 1600 60  0000 C CNN
-F 2 "" H 2100 1350 60  0000 C CNN
-F 3 "" H 2100 1350 60  0000 C CNN
-	1    2050 1300
-	-1   0    0    -1
-$EndComp
 Wire Wire Line
 	3950 1200 2550 1200
@@
 Wire Wire Line
 	3850 1400 3850 1900
-$Comp
-L CONN_2 P?
-U 1 1 52477560
-P 1150 1300
-F 0 "P?" V 1100 1300 40  0000 C CNN
-F 1 "engine_1" V 1200 1300 40  0000 C CNN
-F 2 "~" H 1150 1300 60  0000 C CNN
-F 3 "~" H 1150 1300 60  0000 C CNN
-	1    1150 1300
-	-1   0    0    -1
-$EndComp
 $Comp
 L CONN_2 P?
 U 1 1 5247758D
-P 10000 1250
-F 0 "P?" V 9950 1250 40  0000 C CNN
-F 1 "engine_4" V 10050 1250 40  0000 C CNN
-F 2 "~" H 10000 1250 60  0000 C CNN
-F 3 "~" H 10000 1250 60  0000 C CNN
-	1    10000 1250
-	1    0    0    -1
-$EndComp
-$Comp
-L +12V #PWR?
-U 1 1 524775A2
-P 1450 950
-F 0 "#PWR?" H 1450 900 20  0001 C CNN
-F 1 "+12V" H 1450 1050 30  0000 C CNN
-F 2 "" H 1450 950 60  0000 C CNN
-F 3 "" H 1450 950 60  0000 C CNN
-	1    1450 950
-	1    0    0    -1
-$EndComp
-Wire Wire Line
-	1450 950  1450 1300
-Wire Wire Line
-	1450 1300 1500 1300
+P 10250 1250
+F 0 "P?" V 10200 1250 40  0000 C CNN
+F 1 "engine_4" V 10300 1250 40  0000 C CNN
+F 2 "~" H 10250 1250 60  0000 C CNN
+F 3 "~" H 10250 1250 60  0000 C CNN
+	1    10250 1250
+	1    0    0    -1
+$EndComp
 Wire Wire Line
 	9650 1250 9700 1250
@@
 Wire Wire Line
 	8550 1250 8550 1500
+Text Notes 4400 5200 0    60   ~ 0
+115200 8N1 commands\n
+Text Notes 5900 1350 0    60   ~ 0
+For 2 servo
+$Comp
+L DIODE D?
+U 1 1 524844F0
+P 9750 1550
+F 0 "D?" H 9750 1650 40  0000 C CNN
+F 1 "DIODE" H 9750 1450 40  0000 C CNN
+F 2 "~" H 9750 1550 60  0000 C CNN
+F 3 "~" H 9750 1550 60  0000 C CNN
+	1    9750 1550
+	0    1    -1   0
+$EndComp
+$Comp
+L DIODE D?
+U 1 1 524844FF
+P 9500 1450
+F 0 "D?" H 9500 1550 40  0000 C CNN
+F 1 "DIODE" H 9500 1350 40  0000 C CNN
+F 2 "~" H 9500 1450 60  0000 C CNN
+F 3 "~" H 9500 1450 60  0000 C CNN
+	1    9500 1450
+	0    -1   -1   0
+$EndComp
+$Comp
+L DIODE D?
+U 1 1 5248450E
+P 9500 800
+F 0 "D?" H 9500 900 40  0000 C CNN
+F 1 "DIODE" H 9500 700 40  0000 C CNN
+F 2 "~" H 9500 800 60  0000 C CNN
+F 3 "~" H 9500 800 60  0000 C CNN
+	1    9500 800
+	1    0    0    -1
+$EndComp
+$Comp
+L DIODE D?
+U 1 1 5248451D
+P 9800 950
+F 0 "D?" H 9800 1050 40  0000 C CNN
+F 1 "DIODE" H 9800 850 40  0000 C CNN
+F 2 "~" H 9800 950 60  0000 C CNN
+F 3 "~" H 9800 950 60  0000 C CNN
+	1    9800 950
+	0    1    1    0
+$EndComp
+$Comp
+L STM32F103C8 U1
+U 1 1 52384296
+P 4200 3150
+F 0 "U1" H 3300 4300 60  0000 C CNN
+F 1 "STM32F103C8" H 4150 3400 60  0000 C CNN
+F 2 "" H 4200 3150 60  0000 C CNN
+F 3 "" H 4200 3150 60  0000 C CNN
+	1    4200 3150
+	1    0    0    -1
+$EndComp
+Wire Wire Line
+	9500 1650 9650 1650
+Wire Wire Line
+	9650 1650 9650 1350
 $Comp
 L VSS #PWR?
-U 1 1 524776EE
+U 1 1 524846CF
+P 9750 1750
+F 0 "#PWR?" H 9750 1750 30  0001 C CNN
+F 1 "VSS" H 9750 1680 30  0000 C CNN
+F 2 "" H 9750 1750 60  0000 C CNN
+F 3 "" H 9750 1750 60  0000 C CNN
+	1    9750 1750
+	1    0    0    -1
+$EndComp
+$Comp
+L VSS #PWR?
+U 1 1 5248471E
+P 10050 800
+F 0 "#PWR?" H 10050 800 30  0001 C CNN
+F 1 "VSS" H 10050 730 30  0000 C CNN
+F 2 "" H 10050 800 60  0000 C CNN
+F 3 "" H 10050 800 60  0000 C CNN
+	1    10050 800
+	1    0    0    -1
+$EndComp
+Wire Wire Line
+	9800 750  9800 650
+Wire Wire Line
+	9800 650  10050 650
+Wire Wire Line
+	10050 650  10050 800
+Wire Wire Line
+	9650 1350 9900 1350
+Wire Wire Line
+	9300 800  9300 950
+Wire Wire Line
+	9300 950  9500 950
+Wire Wire Line
+	9500 950  9500 1150
+Wire Wire Line
+	9650 1150 9900 1150
+$Comp
+L +12V #PWR?
+U 1 1 524852D5
+P 1450 800
+F 0 "#PWR?" H 1450 750 20  0001 C CNN
+F 1 "+12V" H 1450 900 30  0000 C CNN
+F 2 "" H 1450 800 60  0000 C CNN
+F 3 "" H 1450 800 60  0000 C CNN
+	1    1450 800
+	-1   0    0    -1
+$EndComp
+$Comp
+L IR4426 KEY?
+U 1 1 524852DD
+P 2050 1300
+F 0 "KEY?" H 2100 1100 60  0000 C CNN
+F 1 "IR4426" H 2050 1600 60  0000 C CNN
+F 2 "" H 2100 1350 60  0000 C CNN
+F 3 "" H 2100 1350 60  0000 C CNN
+	1    2050 1300
+	-1   0    0    -1
+$EndComp
+$Comp
+L CONN_2 P?
+U 1 1 524852E5
+P 900 1300
+F 0 "P?" V 850 1300 40  0000 C CNN
+F 1 "engine_1" V 950 1300 40  0000 C CNN
+F 2 "~" H 900 1300 60  0000 C CNN
+F 3 "~" H 900 1300 60  0000 C CNN
+	1    900  1300
+	-1   0    0    -1
+$EndComp
+Wire Wire Line
+	1500 1300 1450 1300
+Wire Wire Line
+	1450 1300 1450 800
+$Comp
+L VSS #PWR?
+U 1 1 524852ED
 P 2600 1550
 F 0 "#PWR?" H 2600 1550 30  0001 C CNN
@@
 F 3 "" H 2600 1550 60  0000 C CNN
 	1    2600 1550
-	1    0    0    -1
-$EndComp
-Wire Wire Line
-	2550 1300 2600 1300
+	-1   0    0    -1
+$EndComp
 Wire Wire Line
 	2600 1300 2600 1550
-Text Notes 4400 5200 0    60   ~ 0
-115200 8N1 commands\n
-Text Notes 5900 1350 0    60   ~ 0
-For 2 servo
+$Comp
+L DIODE D?
+U 1 1 524852F5
+P 1400 1600
+F 0 "D?" H 1400 1700 40  0000 C CNN
+F 1 "DIODE" H 1400 1500 40  0000 C CNN
+F 2 "~" H 1400 1600 60  0000 C CNN
+F 3 "~" H 1400 1600 60  0000 C CNN
+	1    1400 1600
+	0    -1   -1   0
+$EndComp
+$Comp
+L DIODE D?
+U 1 1 524852FB
+P 1650 1500
+F 0 "D?" H 1650 1600 40  0000 C CNN
+F 1 "DIODE" H 1650 1400 40  0000 C CNN
+F 2 "~" H 1650 1500 60  0000 C CNN
+F 3 "~" H 1650 1500 60  0000 C CNN
+	1    1650 1500
+	0    1    -1   0
+$EndComp
+$Comp
+L DIODE D?
+U 1 1 52485301
+P 1650 850
+F 0 "D?" H 1650 950 40  0000 C CNN
+F 1 "DIODE" H 1650 750 40  0000 C CNN
+F 2 "~" H 1650 850 60  0000 C CNN
+F 3 "~" H 1650 850 60  0000 C CNN
+	1    1650 850
+	-1   0    0    -1
+$EndComp
+$Comp
+L DIODE D?
+U 1 1 52485307
+P 1350 1000
+F 0 "D?" H 1350 1100 40  0000 C CNN
+F 1 "DIODE" H 1350 900 40  0000 C CNN
+F 2 "~" H 1350 1000 60  0000 C CNN
+F 3 "~" H 1350 1000 60  0000 C CNN
+	1    1350 1000
+	0    -1   1    0
+$EndComp
+Wire Wire Line
+	1500 1700 1500 1400
+$Comp
+L VSS #PWR?
+U 1 1 5248530F
+P 1400 1800
+F 0 "#PWR?" H 1400 1800 30  0001 C CNN
+F 1 "VSS" H 1400 1730 30  0000 C CNN
+F 2 "" H 1400 1800 60  0000 C CNN
+F 3 "" H 1400 1800 60  0000 C CNN
+	1    1400 1800
+	-1   0    0    -1
+$EndComp
+$Comp
+L VSS #PWR?
+U 1 1 52485315
+P 1100 850
+F 0 "#PWR?" H 1100 850 30  0001 C CNN
+F 1 "VSS" H 1100 780 30  0000 C CNN
+F 2 "" H 1100 850 60  0000 C CNN
+F 3 "" H 1100 850 60  0000 C CNN
+	1    1100 850
+	-1   0    0    -1
+$EndComp
+Wire Wire Line
+	1350 800  1350 700
+Wire Wire Line
+	1350 700  1100 700
+Wire Wire Line
+	1100 700  1100 850
+Wire Wire Line
+	1500 1400 1250 1400
+Wire Wire Line
+	1850 850  1850 1000
+Wire Wire Line
+	1850 1000 1650 1000
+Wire Wire Line
+	1650 1000 1650 1200
+Wire Wire Line
+	1500 1200 1250 1200
+Wire Wire Line
+	2600 1300 2550 1300
+Wire Wire Line
+	1500 1700 1650 1700
+$Comp
+L VSS #PWR?
+U 1 1 524767CF
+P 2050 6350
+F 0 "#PWR?" H 2050 6350 30  0001 C CNN
+F 1 "VSS" H 2050 6280 30  0000 C CNN
+F 2 "" H 2050 6350 60  0000 C CNN
+F 3 "" H 2050 6350 60  0000 C CNN
+	1    2050 6350
+	1    0    0    -1
+$EndComp
+$Comp
+L IR4426 KEY?
+U 1 1 524767BD
+P 2550 6350
+F 0 "KEY?" H 2600 6150 60  0000 C CNN
+F 1 "IR4426" H 2550 6650 60  0000 C CNN
+F 2 "" H 2600 6400 60  0000 C CNN
+F 3 "" H 2600 6400 60  0000 C CNN
+	1    2550 6350
+	1    0    0    -1
+$EndComp
 $EndSCHEMATC
