File: schem/test.kicad_pcb (KiCad board)
At the start: 2 copper layers, 17 parts, among them P1 CONN_6, U1 STM32F103C8

Commit message: Переделана заново схема, исправлена куча ошибок
Parts:
- removed 8MHz1: CRYSTAL, SM1206
- removed C1: 100nF, SM1206
- removed C2, C3: 20pF, SM1206
- removed JP_BOOT1: BREAKER, SIL-1
- removed JP_BOOT2: BREAKER, SIL-2
- removed P1: CONN_6, SIL-6
- removed R1: 330, SM1206
- removed R2, R3: 10k, SM1206
- removed R4, R5: 510, SM1206
- removed SWD1: CONN_3, SM2010
- removed U1: STM32F103C8, QFN48
- removed reset1: SW_PUSH, SMD403
- removed uart1: CONN1, SIL-3
- removed uart2: CONN2, SIL-3
