File: newschem/netdroid.kicad_pcb (KiCad board)
At the start: 2 copper layers, 43.2 x 84.5 mm, 46 parts, among them U1 STM32F100C4

Commit message: почти нарисовал схкму. Не нашел переходные отверстия. Заебало.
Parts:
- removed SERVO2: CONN_4, SIL-4
- added ADC1: CONN_2, SIL-2, F.Cu at (38.6, 68.8)
- added ADC2: CONN_2, SIL-2, F.Cu at (38.6, 71.5)
- D11, D12, D13, D14, D21, D22, D23, D24, D31, D32, D33, D34, D41, D42, D43, D44: footprint SM0805 -> SM1206
- U1: footprint QFN48 -> LQFP48
- moved D14 86.5 mm to (43.4, 38.8), turned to 180 degrees
- moved D13 86.1 mm to (37.7, 41.8), turned to 270 degrees
- moved D11 80.6 mm to (37.8, 48.0), turned to 90 degrees
- moved D22 79.4 mm to (66.1, 40.1)
- moved D21 75.9 mm to (71.7, 43.0), turned to 270 degrees
- moved D12 75.6 mm to (43.4, 50.7), turned to 180 degrees
- moved C2 74.5 mm to (37.9, 55.0), turned to 180 degrees
- moved C3 72.3 mm to (37.9, 57.6)
- moved ENG2 70.6 mm to (67.2, 46.2), turned to 270 degrees
- moved C1 70.0 mm to (37.1, 60.8), turned to 90 degrees
- moved D23 69.7 mm to (71.8, 49.3), turned to 90 degrees
- moved ENG1 69.4 mm to (42.2, 44.9), turned to 90 degrees
- moved R2 68.5 mm to (49.1, 56.0), turned to 180 degrees
- moved D24 67.8 mm to (66.0, 51.8)
- moved R1 66.9 mm to (37.1, 64.7), turned to 270 degrees
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Connections:
- KEY1 pad 2: N-0000014 -> N-0000029
- KEY1 pad 4: N-0000013 -> N-0000028
- KEY2 pad 2: N-0000032 -> N-0000024
- KEY2 pad 4: N-0000017 -> N-0000031
- KEY3 pad 2: N-0000029 -> N-0000020
- KEY3 pad 4: N-0000030 (its old number) -> N-0000019
- KEY4 pad 2: N-0000031 -> N-000009
- KEY4 pad 4: N-000005 -> N-0000010
- SERVO1 pad 1: N-0000022 -> N-000005
- SERVO1 pad 2: N-0000021 -> N-0000027
- SERVO1 pad 3: N-0000035 -> N-0000026
- SERVO1 pad 4: N-0000034 -> N-0000025
- U1 pad 10: (no net) -> N-0000021
- U1 pad 11: (no net) -> N-0000022
- U1 pad 16: N-0000029 -> N-0000010
- U1 pad 17: N-0000030 (its old number) -> N-000009
- U1 pad 18: N-0000034 -> N-0000019
- U1 pad 19: N-0000035 -> N-0000020
- U1 pad 25: N-0000023 (its old number) -> N-0000025
- U1 pad 26: N-0000024 -> N-0000026
- U1 pad 27: N-0000025 -> N-0000027
- U1 pad 28: N-0000026 -> N-000005
- U1 pad 29: N-0000031 -> (no net)
- U1 pad 32: N-000005 -> (no net)
- U1 pad 39: N-0000021 -> (no net)
- U1 pad 40: N-0000022 -> (no net)
- U1 pad 42: N-0000013 -> N-0000031
- U1 pad 43: N-0000014 -> N-0000024
- U1 pad 45: N-0000017 -> N-0000028
- U1 pad 46: N-0000032 -> N-0000029
Routing:
- net VSS: track 0.00 -> 323.8 mm
- net +12V: track 0.00 -> 45.8 mm
- net N-0000028: track 0.00 -> 28.4 mm
- net N-0000024: track 0.00 -> 26.7 mm
- net N-0000029: track 0.00 -> 25.2 mm
- net N-0000031: track 0.00 -> 23.7 mm
- net N-0000019: track 0.00 -> 22.6 mm
- net N-000009: track 0.00 -> 22.0 mm
- net N-000005: track 0.00 -> 20.3 mm
- net N-0000020: track 0.00 -> 19.8 mm
- net N-0000010: track 0.00 -> 19.4 mm
- net N-0000027: track 0.00 -> 17.4 mm
- net N-0000023: track 0.00 -> 16.8 mm
- net N-0000048: track 0.00 -> 16.4 mm
- net N-0000011: track 0.00 -> 16.2 mm
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Other:
- rule trace_min: 0.254 -> 0.2

Commit message: захуярил схему
Parts:
- added C4: 100nF, SM0805, F.Cu at (54.9, 95.8)
- added C5: 100nF, SM0805, F.Cu at (46.0, 66.8)
- added C6: 100nF, SM0805, F.Cu at (57.3, 72.3)
- added C7: 100nF, SM0805, F.Cu at (47.8, 60.1)
- added C9: 1uF, SMDHD/VF, B.Cu at (67.0, 98.0)
- added P1: CONN_1, SIL-1, F.Cu at (54.1, 51.6)
- added P2: CONN_1, SIL-1, F.Cu at (62.4, 62.4)
- added P3: CONN_1, SIL-1, F.Cu at (60.6, 72.6)
- added P4: CONN_1, SIL-1, F.Cu at (41.8, 68.6)
- added P5: CONN_1, SIL-1, F.Cu at (48.6, 95.8)
- added P6: CONN_1, SIL-1, F.Cu at (42.4, 98.1)
- added P7: CONN_1, SIL-1, F.Cu at (54.7, 38.2)
- added P8: CONN_1, SIL-1, F.Cu at (60.6, 99.4)
- added PWR1: CONN_2, SIL-2, F.Cu at (67.4, 61.4)
- added PWR2: CONN_3, SIL-3, F.Cu at (54.3, 99.4)
- PSWD1, USART1, USART2: value CONN_4 -> CONN_2; footprint SIL-4 -> SIL-2
- moved R6 38.1 mm to (53.0, 93.5)
- moved LED1 38.1 mm to (57.1, 93.5)
- moved USART2 7.90 mm to (48.6, 74.2), turned to 270 degrees
- moved ADC2 6.85 mm to (44.8, 74.3), turned to 90 degrees
- moved ADC1 6.38 mm to (41.8, 74.3), turned to 90 degrees
- moved R3 5.76 mm to (57.3, 74.5), turned to 0 degrees
- moved PSWD1 5.08 mm to (66.0, 66.0), turned to 90 degrees
- moved USART1 3.22 mm to (71.4, 65.9), turned to 90 degrees
- moved SERVO1 1.81 mm to (68.6, 74.3)
- moved R7 1.56 mm to (66.6, 57.3)
- moved LED2 1.55 mm to (71.1, 57.3)
- moved JP_BOOT1 1.32 mm to (56.8, 77.3)
- moved R5 1.14 mm to (57.0, 80.8), turned to 0 degrees
Connections:
- PSWD1 pad 2: VSS -> N-0000026
- U1 pad 12: N-000003 (its old number) -> N-0000017
- U1 pad 13: N-000004 (its old number) -> N-0000016
- U1 pad 30: N-0000011 (its old number) -> N-0000025
- U1 pad 31: N-0000012 (its old number) -> N-0000024
- U1 pad 37: N-000007 (its old number) -> N-0000026
- USART1 pad 1: VSS -> N-0000025
- USART1 pad 2: N-0000011 (its old number) -> N-0000024
- USART2 pad 1: VSS -> N-0000017
- USART2 pad 2: N-000003 (its old number) -> N-0000016
Routing:
- net +12V: track 45.8 -> 247.1 mm
- net VDD: track 5.30 -> 159.4 mm
- net N-0000024: track 0.00 -> 18.6 mm
- net N-0000025: track 0.00 -> 16.8 mm
- net N-0000026: track 0.00 -> 16.7 mm
- net N-0000011 (its old number): track 16.2 -> 0.00 mm
- net N-000003 (its old number): track 13.8 -> 0.00 mm
- net N-0000012 (its old number): track 13.4 -> 0.00 mm
- net N-000004 (its old number): track 12.3 -> 0.00 mm
- net VSS: track 323.8 -> 334.4 mm
- net N-000007 (its old number): track 7.99 -> 0.00 mm
- net N-0000016: track 0.00 -> 7.49 mm
- net N-0000023: track 16.2 -> 9.08 mm
- net N-0000017: track 0.00 -> 5.58 mm
- net N-0000021: track 11.8 -> 7.87 mm
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
Commit message: вроде все
Routing:
- net (no net): track 0.00 -> 37.9 mm
- net N-0000060: track 8.67 -> 13.7 mm
- removed copper zone on B.Cu, net GND
Other:
- board size 43.2 x 84.5 mm -> 49 x 74 mm
Changed lines of the file:
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@@
   (general
     (links 126)
-    (no_connects 1)
-    (area 32.945069 34.215069 76.274931 118.819931)
+    (no_connects 0)
+    (area 30.018989 31.459169 79.122271 105.586531)
     (thickness 1.6002)
-    (drawings 4)
-    (tracks 476)
+    (drawings 7)
+    (tracks 491)
     (zones 0)
     (modules 62)
@@
   )
   (setup
-    (last_trace_width 3)
+    (last_trace_width 1)
     (user_trace_width 0.235)
     (user_trace_width 0.254)
@@
     (via_min_size 0.889)
     (via_min_drill 0.508)
+    (user_via 1 0)
     (uvia_size 0.508)
     (uvia_drill 0.127)
@@
     (visible_elements 7FFFFF9F)
     (pcbplotparams
-      (layerselection 3178497)
-      (usegerberextensions true)
+      (layerselection 32769)
+      (usegerberextensions false)
       (excludeedgelayer true)
       (linewidth 0.150000)
@@
       (outputformat 1)
       (mirror false)
-      (drillshape 1)
+      (drillshape 0)
       (scaleselection 1)
       (outputdirectory ""))
@@
     )
   )
-  (gr_line (start 33.02 34.29) (end 33.02 118.745) (angle 90) (layer Edge.Cuts) (width 0.14986))
-  (gr_line (start 76.2 118.745) (end 76.2 34.29) (angle 90) (layer Edge.Cuts) (width 0.14986))
-  (gr_line (start 76.2 118.745) (end 33.02 118.745) (angle 90) (layer Edge.Cuts) (width 0.14986))
-  (gr_line (start 33.02 34.29) (end 76.2 34.29) (angle 90) (layer Edge.Cuts) (width 0.14986))
+  (gr_line (start 30.09392 105.50906) (end 79.0448 105.50906) (angle 90) (layer Edge.Cuts) (width 0.14986))
+  (gr_line (start 30.09646 104.14762) (end 30.09646 105.5116) (angle 90) (layer Edge.Cuts) (width 0.14986))
+  (gr_line (start 79.0448 104.1146) (end 79.0448 105.5116) (angle 90) (layer Edge.Cuts) (width 0.14986))
+  (gr_line (start 79.04734 104.14) (end 79.04734 104.12476) (angle 90) (layer Edge.Cuts) (width 0.14986))
+  (gr_line (start 30.099 31.5341) (end 30.099 104.14) (angle 90) (layer Edge.Cuts) (width 0.14986))
+  (gr_line (start 79.0448 31.5341) (end 30.099 31.5341) (angle 90) (layer Edge.Cuts) (width 0.14986))
+  (gr_line (start 79.0448 104.14) (end 79.0448 31.5341) (angle 90) (layer Edge.Cuts) (width 0.14986))
+  (segment (start 78.0542 34.47796) (end 73.23074 34.47796) (width 1) (layer Front) (net 0))
+  (segment (start 73.23074 34.47796) (end 73.22312 34.48558) (width 1) (layer Front) (net 0))
+  (segment (start 75.65136 32.63646) (end 75.65136 36.73348) (width 1) (layer Front) (net 0))
+  (segment (start 75.65136 36.73348) (end 75.64374 36.7411) (width 1) (layer Front) (net 0))
+  (segment (start 73.2028 34.4932) (end 78.0796 34.4932) (width 1) (layer Back) (net 0))
+  (segment (start 75.6412 32.6644) (end 75.6412 36.7538) (width 1) (layer Back) (net 0))
+  (segment (start 36.16452 101.6889) (end 31.02864 101.6889) (width 1) (layer Back) (net 0))
+  (segment (start 31.02864 101.6889) (end 31.0134 101.70414) (width 1) (layer Back) (net 0))
+  (segment (start 33.5153 99.23018) (end 33.5153 104.09174) (width 1) (layer Back) (net 0))
+  (segment (start 33.5153 104.09174) (end 33.528 104.10444) (width 1) (layer Back) (net 0))
+  (segment (start 31.0134 101.7016) (end 36.0426 101.7016) (width 1) (layer Front) (net 0))
+  (segment (start 36.0426 101.7016) (end 36.068 101.727) (width 1) (layer Front) (net 0))
+  (segment (start 33.528 99.187) (end 33.528 104.1146) (width 1) (layer Front) (net 0))
   (segment (start 51.7906 99.3648) (end 51.7906 101.5746) (width 1) (layer Front) (net 1))
   (segment (start 73.88098 88.18118) (end 71.91756 88.18118) (width 1) (layer Front) (net 1))
@@
   (segment (start 63.3476 47.41164) (end 67.16268 47.41164) (width 0.5) (layer Front) (net 32))
   (segment (start 67.16268 47.41164) (end 67.2084 47.45736) (width 0.5) (layer Front) (net 32))
+  (segment (start 67.51066 82.02676) (end 67.51066 86.53272) (width 0.5) (layer Front) (net 33))
+  (segment (start 67.51066 86.53272) (end 67.13728 86.9061) (width 0.5) (layer Front) (net 33))
   (segment (start 67.51066 82.02676) (end 70.78726 82.02676) (width 0.5) (layer Front) (net 33))
   (segment (start 70.78726 82.02676) (end 71.99376 83.23326) (width 0.5) (layer Front) (net 33))
@@
   (segment (start 41.76268 61.60008) (end 37.27958 61.60008) (width 0.5) (layer Front) (net 39))
   (segment (start 37.27958 61.60008) (end 37.12464 61.75502) (width 0.5) (layer Front) (net 39))
-  (segment (start 48.641 95.758) (end 56.90108 95.758) (width 3) (layer Back) (net 40) (status 400000))
+  (segment (start 48.641 95.758) (end 56.90108 95.758) (width 3) (layer Back) (net 40))
   (segment (start 58.17108 94.488) (end 61.468 94.488) (width 3) (layer Back) (net 40))
   (segment (start 56.90108 95.758) (end 58.17108 94.488) (width 3) (layer Back) (net 40))
-  (segment (start 60.59424 72.64908) (end 60.59424 73.2536) (width 3) (layer Back) (net 40) (status C00000))
-  (segment (start 60.59424 73.2536) (end 61.468 74.12736) (width 3) (layer Back) (net 40) (status 400000))
+  (segment (start 60.59424 72.64908) (end 60.59424 73.2536) (width 3) (layer Back) (net 40))
+  (segment (start 60.59424 73.2536) (end 61.468 74.12736) (width 3) (layer Back) (net 40))
   (segment (start 61.468 74.12736) (end 61.468 94.488) (width 3) (layer Back) (net 40))
-  (segment (start 62.4332 62.4332) (end 62.4332 70.5358) (width 3) (layer Back) (net 40) (status 400000))
-  (segment (start 60.31992 72.64908) (end 60.59424 72.64908) (width 3) (layer Back) (net 40) (status C00000))
-  (segment (start 62.4332 70.5358) (end 60.31992 72.64908) (width 3) (layer Back) (net 40) (status 800000))
-  (segment (start 62.4332 62.4332) (end 62.4332 55.5371) (width 3) (layer Back) (net 40) (status 400000))
-  (segment (start 58.48096 51.58486) (end 54.14518 51.58486) (width 3) (layer Back) (net 40) (status 800000))
+  (segment (start 62.4332 62.4332) (end 62.4332 70.5358) (width 3) (layer Back) (net 40))
+  (segment (start 60.31992 72.64908) (end 60.59424 72.64908) (width 3) (layer Back) (net 40))
+  (segment (start 62.4332 70.5358) (end 60.31992 72.64908) (width 3) (layer Back) (net 40))
+  (segment (start 62.4332 62.4332) (end 62.4332 55.5371) (width 3) (layer Back) (net 40))
+  (segment (start 58.48096 51.58486) (end 54.14518 51.58486) (width 3) (layer Back) (net 40))
   (segment (start 62.4332 55.5371) (end 58.48096 51.58486) (width 3) (layer Back) (net 40))
   (segment (start 61.468 94.488) (end 61.4934 94.488) (width 3) (layer Back) (net 40))
@@
   (segment (start 37.12464 59.85002) (end 34.6583 59.85002) (width 0.5) (layer Front) (net 41))
   (segment (start 60.579 82.02676) (end 64.20866 82.02676) (width 1) (layer Front) (net 41))
-  (zone (net -1) (net_name GND) (layer Back) (hatch edge 0.508)
-    (connect_pads (clearance 0.508))
-    (min_thickness 0.254)
-    (fill (arc_segments 16) (thermal_gap 0.508) (thermal_bridge_width 0.889))
-    (polygon
-      (pts
-        (xy 76.073 118.618) (xy 33.147 118.618) (xy 33.147 34.417) (xy 76.073 34.417)
-      )
-    )
-  )
 )

Commit message: Надеюсь, это финальная версия
Parts:
- 8MHz1: footprint SIL-2 -> HC-49V
- moved ADC2 21.3 mm to (27.4, 62.2)
- moved D24 17.3 mm to (54.3, 39.2)
- moved D43 17.3 mm to (25.5, 71.1)
- moved ENG3 17.3 mm to (55.4, 75.6)
- moved R7 17.3 mm to (54.9, 44.7)
- moved KEY3 17.3 mm to (48.5, 74.9)
- moved R2 17.3 mm to (37.3, 43.4)
- moved R5 17.3 mm to (45.2, 68.2)
- moved U1 17.3 mm to (42.4, 53.1)
- moved C9 17.3 mm to (55.2, 85.4)
- moved C7 17.3 mm to (36.1, 47.5)
- moved D11 17.3 mm to (26.0, 35.4)
- moved D12 17.3 mm to (31.6, 38.1)
- moved D13 17.3 mm to (26.0, 29.2)
- moved D14 17.3 mm to (31.6, 26.2)
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Routing:
- net VDD: track 159.4 -> 148.5 mm
- net N-0000021: track 7.87 -> 16.7 mm
- net N-0000017: track 5.58 -> 9.80 mm
- net N-0000039: track 15.7 -> 11.9 mm
- net N-0000061: track 17.5 -> 19.5 mm
- net N-0000020: track 11.3 -> 13.0 mm
- net +12V: track 247.1 -> 248.3 mm
- net N-0000011: track 18.4 -> 19.7 mm
- net N-0000012: track 9.51 -> 10.6 mm
- net N-0000014: track 15.7 -> 16.5 mm
- net N-000008: track 19.4 -> 18.6 mm
- net N-000001: track 23.7 -> 22.9 mm
- net N-0000013: track 12.6 -> 13.2 mm
- net N-000007: track 22.0 -> 21.3 mm
- net N-0000025: track 16.8 -> 17.4 mm

Commit message: заел на будущее
Connections:
- R7 pad 1: N-0000015 (its old number) -> N-0000031
- U1 pad 38: N-0000015 (its old number) -> (no net)
- U1 pad 41: (no net) -> N-0000031
Routing:
- net N-0000031: track 0.00 -> 13.0 mm
- net N-0000015 (its old number): track 11.9 -> 0.00 mm
