File: newschem/netdroid.sch (KiCad schematic (older format))
At the start: 46 parts, among them U1 STM32F100C4

Commit message: Переделана заново схема, исправлена куча ошибок
Parts:
- renumbered D7 to D11, D2 to D12, D8 to D13, D4 to D14, D5 to D21, D1 to D22, D6 to D23, D3 to D24, D11 to D31, D16 to D32, D12 to D33, D15 to D34, D13 to D41, D18 to D42, D14 to D43, D17 to D44, D9 to LED1, D10 to LED2
Connections:
- net labels removed: +3.3V
- wire segments 124 -> 133
Other:
- moved on the sheet: D11, D12, D13, D14, D21, D22, D23, D24, ENG1, ENG2, ENG3, ENG4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

Commit message: почти нарисовал схкму. Не нашел переходные отверстия. Заебало.
Parts:
- removed SERVO1: CONN_4, symbol CONN_4
- added ADC1, ADC2: CONN_2, symbol CONN_2
- renumbered SERVO2 to SERVO1
Changed lines of the file:
@@
 LIBS:contrib
 LIBS:valves
+LIBS:netdroid-cache
 EELAYER 27 0
 EELAYER END
@@
 Sheet 1 1
 Title "WebDroid  Neuraxis"
-Date "22 oct 2013"
+Date "7 nov 2013"
 Rev ""
 Comp "BSUIR 2013"
@@
 L VSS #PWR01
 U 1 1 52384A32
-P 3000 4350
-F 0 "#PWR01" H 3000 4350 30  0001 C CNN
-F 1 "VSS" H 3000 4280 30  0000 C CNN
-F 2 "" H 3000 4350 60  0000 C CNN
-F 3 "" H 3000 4350 60  0000 C CNN
-	1    3000 4350
+P 2950 4350
+F 0 "#PWR01" H 2950 4350 30  0001 C CNN
+F 1 "VSS" H 2950 4280 30  0000 C CNN
+F 2 "" H 2950 4350 60  0000 C CNN
+F 3 "" H 2950 4350 60  0000 C CNN
+	1    2950 4350
 	0    1    -1   0
 $EndComp
@@
 L VDD #PWR029
 U 1 1 525D1128
-P 5900 7500
-F 0 "#PWR029" H 5900 7600 30  0001 C CNN
-F 1 "VDD" H 5900 7610 30  0000 C CNN
-F 2 "" H 5900 7500 60  0000 C CNN
-F 3 "" H 5900 7500 60  0000 C CNN
-	1    5900 7500
+P 5800 7500
+F 0 "#PWR029" H 5800 7600 30  0001 C CNN
+F 1 "VDD" H 5800 7610 30  0000 C CNN
+F 2 "" H 5800 7500 60  0000 C CNN
+F 3 "" H 5800 7500 60  0000 C CNN
+	1    5800 7500
 	1    0    0    -1
 $EndComp
@@
 L VSS #PWR031
 U 1 1 525D1156
-P 9350 5550
-F 0 "#PWR031" H 9350 5550 30  0001 C CNN
-F 1 "VSS" H 9350 5480 30  0000 C CNN
-F 2 "" H 9350 5550 60  0000 C CNN
-F 3 "" H 9350 5550 60  0000 C CNN
-	1    9350 5550
+P 9400 5550
+F 0 "#PWR031" H 9400 5550 30  0001 C CNN
+F 1 "VSS" H 9400 5480 30  0000 C CNN
+F 2 "" H 9400 5550 60  0000 C CNN
+F 3 "" H 9400 5550 60  0000 C CNN
+	1    9400 5550
 	0    -1   -1   0
 $EndComp
@@
 $EndComp
 $Comp
-L CONN_4 SERVO2
+L CONN_4 SERVO1
 U 1 1 525D363D
 P 4450 7450
-F 0 "SERVO2" V 4400 7450 50  0000 C CNN
+F 0 "SERVO1" V 4400 7450 50  0000 C CNN
 F 1 "CONN_4" V 4500 7450 50  0000 C CNN
 F 2 "" H 4450 7450 60  0000 C CNN
 F 3 "" H 4450 7450 60  0000 C CNN
 	1    4450 7450
-	0    1    1    0
-$EndComp
-$Comp
-L CONN_4 SERVO1
-U 1 1 525D3652
-P 3950 7450
-F 0 "SERVO1" V 3900 7450 50  0000 C CNN
-F 1 "CONN_4" V 4000 7450 50  0000 C CNN
-F 2 "" H 3950 7450 60  0000 C CNN
-F 3 "" H 3950 7450 60  0000 C CNN
-	1    3950 7450
 	0    1    1    0
 $EndComp
@@
 	3050 4250 3050 4450
 Wire Wire Line
-	3050 4350 3000 4350
+	2950 4350 3050 4350
 Connection ~ 3050 4350
 Wire Wire Line
@@
 	2750 7550 2600 7550
 Wire Wire Line
-	3150 5750 4700 5750
-Wire Wire Line
-	3250 5850 4700 5850
-Wire Wire Line
 	8450 2750 8600 2750
 Wire Wire Line
@@
 	9650 1400 9450 1400
 Wire Wire Line
-	9650 850  9650 1400
+	9650 750  9650 1400
 Wire Wire Line
 	8550 1400 8500 1400
@@
 	9450 1300 9850 1300
 Wire Wire Line
-	8250 1500 8550 1500
-Wire Wire Line
-	8150 1300 8550 1300
-Wire Wire Line
-	8450 2750 8450 4950
-Wire Wire Line
-	8450 4950 7700 4950
-Wire Wire Line
-	8350 2550 8350 4650
-Wire Wire Line
-	8350 4650 7700 4650
-Wire Wire Line
-	8250 1500 8250 4550
-Wire Wire Line
-	8250 4550 7700 4550
-Wire Wire Line
-	8150 1300 8150 4450
-Wire Wire Line
-	8150 4450 7700 4450
+	4450 1500 8550 1500
+Wire Wire Line
+	4200 1300 8550 1300
 Wire Wire Line
 	7700 5350 8450 5350
@@
 Wire Wire Line
 	4300 6150 4300 7100
-Wire Wire Line
-	4700 5350 4100 5350
-Wire Wire Line
-	4100 5350 4100 7100
-Wire Wire Line
-	4700 5250 4000 5250
-Wire Wire Line
-	4000 5250 4000 7100
-Wire Wire Line
-	4700 5050 3900 5050
-Wire Wire Line
-	3900 5050 3900 7100
-Wire Wire Line
-	4700 4950 3800 4950
-Wire Wire Line
-	3800 4950 3800 7100
 Connection ~ 9650 2550
 Connection ~ 9600 1300
@@
 Connection ~ 9750 1300
 Wire Wire Line
-	3250 5850 3250 6450
-Wire Wire Line
 	3250 6450 1650 6450
 Wire Wire Line
@@
 	1650 7050 1700 7050
 Wire Wire Line
-	3150 5750 3150 6350
+	3150 5550 3150 6350
 Wire Wire Line
 	3150 6350 1550 6350
@@
 	3700 5150 4700 5150
 Wire Wire Line
-	4700 5550 3250 5550
-Wire Wire Line
-	4700 5650 3150 5650
-Wire Wire Line
 	3700 4900 3700 5150
 Wire Wire Line
 	1200 4700 1200 4900
 Wire Wire Line
-	3150 5650 3150 5100
-Wire Wire Line
-	3150 5100 1200 5100
+	1200 5100 3450 5100
 Wire Wire Line
 	1200 5100 1200 5650
@@
 	1200 5650 1250 5650
 Wire Wire Line
-	3250 5550 3250 5000
-Wire Wire Line
-	3250 5000 1100 5000
+	1100 5000 3550 5000
 Wire Wire Line
 	1100 5000 1100 5850
@@
 L +12V #PWR034
 U 1 1 52665274
-P 9650 850
-F 0 "#PWR034" H 9650 800 20  0001 C CNN
-F 1 "+12V" H 9650 950 30  0000 C CNN
-F 2 "" H 9650 850 60  0000 C CNN
-F 3 "" H 9650 850 60  0000 C CNN
-	1    9650 850
+P 9650 750
+F 0 "#PWR034" H 9650 700 20  0001 C CNN
+F 1 "+12V" H 9650 850 30  0000 C CNN
+F 2 "" H 9650 750 60  0000 C CNN
+F 3 "" H 9650 750 60  0000 C CNN
+	1    9650 750
 	1    0    0    -1
 $EndComp
@@
 	1    0    0    -1
 $EndComp
-Connection ~ 9650 850
 Connection ~ 9750 3150
 Connection ~ 2400 6250
 Connection ~ 2800 6650
 Connection ~ 4000 3350
+Wire Wire Line
+	3450 5100 3450 5850
+Wire Wire Line
+	3550 5000 3550 5750
+Wire Wire Line
+	3550 5750 4700 5750
+Wire Wire Line
+	3450 5850 4700 5850
+Wire Wire Line
+	3150 5550 4700 5550
+Wire Wire Line
+	3250 6450 3250 5650
+Wire Wire Line
+	3250 5650 4700 5650
+Wire Wire Line
+	7700 4450 8450 4450
+Wire Wire Line
+	8350 4550 7700 4550
+Wire Wire Line
+	8350 4550 8350 2550
+Wire Wire Line
+	8450 4450 8450 2750
+$Comp
+L CONN_2 ADC2
+U 1 1 527B57AD
+P 7800 2350
+F 0 "ADC2" V 7750 2350 40  0000 C CNN
+F 1 "CONN_2" V 7850 2350 40  0000 C CNN
+F 2 "" H 7800 2350 60  0000 C CNN
+F 3 "" H 7800 2350 60  0000 C CNN
+	1    7800 2350
+	0    -1   -1   0
+$EndComp
+$Comp
+L CONN_2 ADC1
+U 1 1 527B57C9
+P 7300 2350
+F 0 "ADC1" V 7250 2350 40  0000 C CNN
+F 1 "CONN_2" V 7350 2350 40  0000 C CNN
+F 2 "" H 7300 2350 60  0000 C CNN
+F 3 "" H 7300 2350 60  0000 C CNN
+	1    7300 2350
+	0    -1   -1   0
+$EndComp
+$Comp
+L VSS #PWR042
+U 1 1 527B57D1
+P 7200 2700
+F 0 "#PWR042" H 7200 2700 30  0001 C CNN
+F 1 "VSS" H 7200 2630 30  0000 C CNN
+F 2 "" H 7200 2700 60  0000 C CNN
+F 3 "" H 7200 2700 60  0000 C CNN
+	1    7200 2700
+	1    0    0    -1
+$EndComp
+$Comp
+L VSS #PWR043
+U 1 1 527B57E0
+P 7700 2700
+F 0 "#PWR043" H 7700 2700 30  0001 C CNN
+F 1 "VSS" H 7700 2630 30  0000 C CNN
+F 2 "" H 7700 2700 60  0000 C CNN
+F 3 "" H 7700 2700 60  0000 C CNN
+	1    7700 2700
+	1    0    0    -1
+$EndComp
+Wire Wire Line
+	7700 3950 7900 3950
+Wire Wire Line
+	7900 3950 7900 2700
+Wire Wire Line
+	7700 3850 7800 3850
+Wire Wire Line
+	7800 3850 7800 2850
+Wire Wire Line
+	7800 2850 7400 2850
+Wire Wire Line
+	7400 2850 7400 2700
+Wire Wire Line
+	9350 5550 9400 5550
+Wire Wire Line
+	5900 7500 5800 7500
+Wire Wire Line
+	4200 1300 4200 5050
+Wire Wire Line
+	4200 5050 4700 5050
+Wire Wire Line
+	4450 1500 4450 4950
+Wire Wire Line
+	4450 4950 4700 4950
 $EndSCHEMATC

Commit message: захуярил схему
Parts:
- removed PSWD1, USART1, USART2: CONN_4, symbol CONN_4
- added C4, C5, C6, C7: 100nF, ~, symbol CSMALL
- added C9: 1uF, ~, symbol CSMALL
- added P1, P2, P3, P4, P5, P6, P7, P8: CONN_1, symbol CONN_1
- added PSWD1, PWR1, USART1, USART2: CONN_2, symbol CONN_2
- added PWR2: CONN_3, symbol CONN_3
Connections:
- wire segments 133 -> 141

Commit message: заел на будущее
Connections:
- wire segments 141 -> 139
Other:
- moved on the sheet: LED2, R7
Changed lines of the file:
@@
 Sheet 1 1
 Title "WebDroid  Neuraxis"
-Date "11 nov 2013"
+Date "19 nov 2013"
 Rev ""
 Comp "BSUIR 2013"
@@
 L LED LED2
 U 1 1 525D114A
-P 9150 5550
-F 0 "LED2" H 9150 5650 50  0000 C CNN
-F 1 "LED" H 9150 5450 50  0000 C CNN
-F 2 "~" H 9150 5550 60  0000 C CNN
-F 3 "~" H 9150 5550 60  0000 C CNN
-	1    9150 5550
-	1    0    0    -1
+P 4000 5450
+F 0 "LED2" H 4000 5550 50  0000 C CNN
+F 1 "LED" H 4000 5350 50  0000 C CNN
+F 2 "~" H 4000 5450 60  0000 C CNN
+F 3 "~" H 4000 5450 60  0000 C CNN
+	1    4000 5450
+	-1   0    0    1
 $EndComp
 $Comp
 L R R7
 U 1 1 525D1150
-P 8700 5550
-F 0 "R7" V 8780 5550 40  0000 C CNN
-F 1 "R" V 8707 5551 40  0000 C CNN
-F 2 "~" V 8630 5550 30  0000 C CNN
-F 3 "~" H 8700 5550 30  0000 C CNN
-	1    8700 5550
-	0    -1   -1   0
+P 4450 5450
+F 0 "R7" V 4530 5450 40  0000 C CNN
+F 1 "R" V 4457 5451 40  0000 C CNN
+F 2 "~" V 4380 5450 30  0000 C CNN
+F 3 "~" H 4450 5450 30  0000 C CNN
+	1    4450 5450
+	0    1    1    0
 $EndComp
 $Comp
 L VSS #PWR54
 U 1 1 525D1156
-P 9400 5550
-F 0 "#PWR54" H 9400 5550 30  0001 C CNN
-F 1 "VSS" H 9400 5480 30  0000 C CNN
-F 2 "" H 9400 5550 60  0000 C CNN
-F 3 "" H 9400 5550 60  0000 C CNN
-	1    9400 5550
-	0    -1   -1   0
+P 3750 5450
+F 0 "#PWR54" H 3750 5450 30  0001 C CNN
+F 1 "VSS" H 3750 5380 30  0000 C CNN
+F 2 "" H 3750 5450 60  0000 C CNN
+F 3 "" H 3750 5450 60  0000 C CNN
+	1    3750 5450
+	0    1    1    0
 $EndComp
 $Comp
@@
 Wire Wire Line
 	4200 1300 8550 1300
-Wire Wire Line
-	7700 5350 8450 5350
-Wire Wire Line
-	8450 5350 8450 5550
 Wire Wire Line
 	7700 5250 8750 5250
@@
 	7400 2850 7400 2700
 Wire Wire Line
-	9350 5550 9400 5550
+	3800 5450 3750 5450
 Wire Wire Line
 	5900 7500 5800 7500

Commit message: PWM init/control implemented
Parts:
- renumbered ENG2 to ENG1, ENG1 to ENG2, ENG4 to ENG3, ENG3 to ENG4
Changed lines of the file:
@@
 Sheet 1 1
 Title "WebDroid  Neuraxis"
-Date "19 nov 2013"
+Date "26 nov 2013"
 Rev ""
 Comp "BSUIR 2013"
@@
 $EndComp
 $Comp
-L CONN_2 ENG3
+L CONN_2 ENG4
 U 1 1 5247758D
 P 10200 1400
-F 0 "ENG3" V 10150 1400 40  0000 C CNN
+F 0 "ENG4" V 10150 1400 40  0000 C CNN
 F 1 "engpin" V 10250 1400 40  0000 C CNN
 F 2 "~" H 10200 1400 60  0000 C CNN
@@
 $EndComp
 $Comp
-L CONN_2 ENG1
+L CONN_2 ENG2
 U 1 1 524852E5
 P 2900 5750
-F 0 "ENG1" V 2850 5750 40  0000 C CNN
+F 0 "ENG2" V 2850 5750 40  0000 C CNN
 F 1 "engpin" V 2950 5750 40  0000 C CNN
 F 2 "~" H 2900 5750 60  0000 C CNN
@@
 $EndComp
 $Comp
-L CONN_2 ENG2
+L CONN_2 ENG1
 U 1 1 525D046A
 P 3350 7150
-F 0 "ENG2" V 3300 7150 40  0000 C CNN
+F 0 "ENG1" V 3300 7150 40  0000 C CNN
 F 1 "engpin" V 3400 7150 40  0000 C CNN
 F 2 "~" H 3350 7150 60  0000 C CNN
@@
 $EndComp
 $Comp
-L CONN_2 ENG4
+L CONN_2 ENG3
 U 1 1 525D0888
 P 10250 2650
-F 0 "ENG4" V 10200 2650 40  0000 C CNN
+F 0 "ENG3" V 10200 2650 40  0000 C CNN
 F 1 "engpin" V 10300 2650 40  0000 C CNN
 F 2 "~" H 10250 2650 60  0000 C CNN
